File: macropadv2/macropadv2.kicad_pcb (KiCad board)
At the start: 2 copper layers, 57.8 x 87 mm, 37 parts, among them J1 USB4085-GF-A_REVA, SW1 SW_SPST, SW10 SW_SPST, SW11 SW_SPST, SW12 SW_SPST, SW13 SW_Push, SW2 SW_SPST, SW3 SW_SPST, SW4 SW_SPST, SW5 SW_SPST, SW6 SW_SPST, SW7 SW_SPST, SW8 SW_SPST, SW9 SW_SPST, U1 ATMEGA32U2

Commit message: added encoder
Parts:
- added C5: 0.1uF, Capacitor_SMD:C_0603_1608Metric, B.Cu at (118.0, 60.2)
- added C6: 10uF, Capacitor_SMD:C_0603_1608Metric, B.Cu at (118.0, 64.8)
- added D13: D_Small, keyboard_parts:D_SOD123W_hand, B.Cu at (157.5, 118.5)
- added D14: D_Small, keyboard_parts:D_SOD123W_hand, B.Cu at (138.5, 118.5)
- added D15: D_Small, keyboard_parts:D_SOD123W_hand, B.Cu at (119.2, 118.2)
- added D16: D_Small, keyboard_parts:D_SOD123W_hand, B.Cu at (100.2, 118.2)
- added R10: 10k, Resistor_SMD:R_0603_1608Metric_Pad0.98x0.95mm_HandSolder, B.Cu at (111.0, 67.5)
- added R7: 22, Resistor_SMD:R_0603_1608Metric_Pad0.98x0.95mm_HandSolder, F.Cu at (131.9, 45.2)
- added R8: 22, Resistor_SMD:R_0603_1608Metric_Pad0.98x0.95mm_HandSolder, F.Cu at (135.7, 45.2)
- added R9: 10k, Resistor_SMD:R_0603_1608Metric_Pad0.98x0.95mm_HandSolder, B.Cu at (133.0, 64.5)
- added SW14: SW_SPST, keyswitches_2:Kailh_socket_MX, F.Cu at (133.3, 114.3)
- added SW15: SW_SPST, keyswitches_2:Kailh_socket_MX, F.Cu at (114.3, 114.3)
- added SW16: SW_SPST, keyswitches_2:Kailh_socket_MX, F.Cu at (95.2, 114.3)
- added SW17: SW_Push, Button_Switch_SMD:SW_SPST_TL3342, B.Cu at (127.8, 63.5)
- C1: value 1uF -> 10nF; footprint keyboard_parts:C_1608 -> Capacitor_SMD:C_0603_1608Metric
- C2: value 0.1uF -> 10nF; footprint keyboard_parts:C_1608 -> Capacitor_SMD:C_0603_1608Metric
- C3: value 0.1uF -> 1uF; footprint keyboard_parts:C_1608 -> Capacitor_SMD:C_0603_1608Metric
- C4: value 10uF -> 0.1uF; footprint keyboard_parts:C_1608 -> Capacitor_SMD:C_0603_1608Metric
- R3, R4: value 22 -> 10k
- R5, R6: moved to F.Cu
- SW13: value SW_Push -> SW_SPST; footprint Button_Switch_SMD:SW_SPST_TL3342 -> keyswitches_2:Kailh_socket_MX; moved to F.Cu
- SW4: value SW_SPST -> RotaryEncoder_Switch; footprint keyswitches_2:Kailh_socket_MX -> Encoder:PEC11L
- U1: footprint keyboard_parts:QFP32 -> Package_DFN_QFN:VQFN-32-1EP_5x5mm_P0.5mm_EP3.15x3.15mm
- moved D4 97.3 mm to (97.8, 54.2), turned to 90 degrees
- moved SW4 92.5 mm to (95.2, 57.1)
- moved SW7 75.7 mm to (114.3, 76.2)
- moved SW8 75.7 mm to (95.2, 76.2)
- moved D8 75.1 mm to (100.2, 80.2), turned to 90 degrees
- moved D7 75.0 mm to (119.4, 80.2), turned to 90 degrees
- moved C2 69.5 mm to (91.2, 60.8)
- moved R4 69.2 mm to (91.2, 62.5)
- moved C1 65.7 mm to (98.8, 60.8)
- moved R3 61.5 mm to (98.8, 62.5), turned to 180 degrees
- moved SW10 60.3 mm to (133.3, 95.2)
- moved SW12 60.3 mm to (95.2, 95.2)
- moved SW11 60.3 mm to (114.3, 95.2)
- moved R6 59.9 mm to (121.8, 35.2)
- moved D12 59.5 mm to (100.2, 99.2), turned to 90 degrees
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Connections:
- C1 pad 1: GND -> Net-(C1-Pad1)
- C1 pad 2: Net-(C1-Pad2) -> GND
- C2 pad 2: VCC -> Net-(C2-Pad2)
- C3 pad 2: VCC -> Net-(C3-Pad2)
- D10 pad 1: /row3 -> /row2
- D11 pad 1: /row3 -> /row2
- D12 pad 1: /row3 -> /row2
- D4 pad 1: /row1 -> /row0
- D7 pad 1: /row2 -> /row1
- D8 pad 1: /row2 -> /row1
- J1 pad A8: Net-(J1-PadA8) -> unconnected-(J1-PadA8)
- J1 pad B8: Net-(J1-PadB8) -> unconnected-(J1-PadB8)
- R1 pad 1: /CC1 -> VCC
- R1 pad 2: GND -> Net-(C1-Pad1)
- R2 pad 1: /CC2 -> VCC
- R2 pad 2: GND -> Net-(C2-Pad2)
- R3 pad 1: /D- -> /ENC_A
- R3 pad 2: /D_P -> Net-(C1-Pad1)
- R4 pad 1: /D+ -> /ENC_B
- R4 pad 2: /D_N -> Net-(C2-Pad2)
- R5 pad 1: Net-(R5-Pad1) -> /CC1
- R5 pad 2: VCC -> GND
- R6 pad 1: Net-(R6-Pad1) -> /CC2
- SW10 pad 2: /col0 -> /col1
- SW11 pad 2: /col1 -> /col2
- SW12 pad 2: /col2 -> /col3
- SW13 pad 1: Net-(R5-Pad1) -> Net-(D13-Pad2)
- SW13 pad 2: GND -> /col0
- SW5 pad 2: /col1 -> /col0
- SW6 pad 2: /col2 -> /col1
- SW7 pad 2: /col0 -> /col2
- SW8 pad 2: /col1 -> /col3
- SW9 pad 2: /col2 -> /col0
- U1 pad 1: Net-(U1-Pad1) -> unconnected-(U1-Pad1)
- U1 pad 10: Net-(U1-Pad10) -> unconnected-(U1-Pad10)
- U1 pad 11: Net-(U1-Pad11) -> unconnected-(U1-Pad11)
- U1 pad 12: Net-(U1-Pad12) -> unconnected-(U1-Pad12)
- U1 pad 13: Net-(R6-Pad1) -> Net-(R10-Pad1)
- U1 pad 14: Net-(U1-Pad14) -> unconnected-(U1-Pad14)
- U1 pad 15: Net-(U1-Pad15) -> unconnected-(U1-Pad15)
- U1 pad 16: Net-(U1-Pad16) -> unconnected-(U1-Pad16)
- U1 pad 2: Net-(U1-Pad2) -> unconnected-(U1-Pad2)
- U1 pad 22: Net-(U1-Pad22) -> unconnected-(U1-Pad22)
- U1 pad 23: Net-(U1-Pad23) -> unconnected-(U1-Pad23)
- U1 pad 24: Net-(R5-Pad1) -> Net-(R9-Pad1)
- U1 pad 25: Net-(U1-Pad25) -> unconnected-(U1-Pad25)
- U1 pad 27: Net-(C1-Pad2) -> Net-(C3-Pad2)
- U1 pad 29: /D_N -> /D_P
- U1 pad 30: /D_P -> /D_N
- U1 pad 5: Net-(U1-Pad5) -> unconnected-(U1-Pad5)
- U1 pad 6: Net-(U1-Pad6) -> /ENC_A
- U1 pad 7: Net-(U1-Pad7) -> /ENC_B
- U1 pad 8: Net-(U1-Pad8) -> unconnected-(U1-Pad8)
- U1 pad 9: Net-(U1-Pad9) -> unconnected-(U1-Pad9)
Routing:
- net /row2: track 95.1 -> 0.00 mm, vias 2 -> 0
- net /col2: track 94.5 -> 0.00 mm
- net /col1: track 85.2 -> 0.00 mm, vias 7 -> 0
- net /row1: track 76.5 -> 0.00 mm, vias 2 -> 0
- net /col0: track 69.1 -> 0.00 mm, vias 6 -> 0
- net /row0: track 58.1 -> 0.00 mm
- net VCC: track 51.4 -> 0.00 mm
- net /row3: track 39.8 -> 0.00 mm
- net /D+: track 26.8 -> 0.00 mm, vias 1 -> 0
- net Net-(R5-Pad1): track 26.4 -> 0.00 mm
- net /D-: track 25.5 -> 0.00 mm
- net GND: track 15.6 -> 0.00 mm, vias 4 -> 0
- net Net-(D10-Pad2): track 9.29 -> 0.00 mm
- net Net-(D12-Pad2): track 8.90 -> 0.00 mm
- net Net-(D6-Pad2): track 8.90 -> 0.00 mm
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- removed copper zone on B.Cu, net GND
Other:
- board outline removed
- net class Default removed
